File: Hardware/AldervendAdapter/AldervendAdapter.kicad_pcb (KiCad board)
At the start: 2 copper layers, 85 x 60 mm, 42 parts, among them J101 MDB_MASTER, J102 MDB_SLAVE, J103 PROG, SW101 RESET, SW102 BOOT, U101 PC817, U102 PC817, U103 K7805M-1000R3, U104 AMS1117-3.3, U106 ESP32-C6-MINI-1

Commit message: Last style
Parts:
- C101: footprint Capacitor_SMD:C_Elec_5x5.4 -> Capacitor_SMD:CP_Elec_6.3x5.4
- moved C101 2.98 mm to (198.5, 81.5)
Routing:
- net +36V: track 37.6 -> 41.4 mm
- net Earth: vias 9 -> 11
Changed lines of the file:
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@@
 		(tags "resistor")
 		(property "Reference" "R104"
-			(at -3.5 0 0)
+			(at 0 -2 0)
 			(layer "F.SilkS")
 			(effects
@@
 			)
 		)
-		(property "LSCS#" ""
+		(property "LSCS#" "C114098"
 			(at 0 0 270)
 			(unlocked yes)
@@
 		)
 	)
-	(footprint "Capacitor_SMD:C_Elec_5x5.4"
+	(footprint "Capacitor_SMD:CP_Elec_6.3x5.4"
 		(layer "F.Cu")
-		(at 201.4375 81 180)
-		(descr "SMD capacitor, aluminum electrolytic nonpolar, 5.0x5.4mm")
-		(tags "capacitor electrolytic nonpolar")
+		(at 198.5 81.5 180)
+		(descr "SMD capacitor, aluminum electrolytic, Panasonic C55, 6.3x5.4mm")
+		(tags "capacitor electrolytic")
 		(property "Reference" "C101"
-			(at 0.4375 -3.7 0)
+			(at 0 -4.35 180)
 			(layer "F.SilkS")
 			(effects
@@
 		)
 		(property "Value" "33uF"
-			(at 0 3.7 0)
+			(at 0 4.35 180)
 			(layer "F.Fab")
 			(effects
@@
 		)
 		(property "Datasheet" "~"
-			(at 0 0 0)
+			(at 0 0 180)
 			(layer "F.Fab")
 			(hide yes)
@@
 		)
 		(property "Description" "Polarized capacitor, small symbol"
-			(at 0 0 0)
+			(at 0 0 180)
 			(layer "F.Fab")
 			(hide yes)
@@
 		(attr smd)
 		(fp_line
-			(start 2.76 2.76)
-			(end 2.76 1.06)
+			(start 3.41 3.41)
+			(end 3.41 1.06)
+			(stroke
+				(width 0.12)
+				(type solid)
+			)
+			(layer "F.SilkS")
+		)
+		(fp_line
+			(start 3.41 -3.41)
+			(end 3.41 -1.06)
+			(stroke
+				(width 0.12)
+				(type solid)
+			)
+			(layer "F.SilkS")
+		)
+		(fp_line
+			(start -2.345563 3.41)
+			(end 3.41 3.41)
 			(stroke
 				(width 0.12)
@@
 		)
 		(fp_line
-			(start 2.76 -2.76)
-			(end 2.76 -1.06)
+			(start -2.345563 -3.41)
+			(end 3.41 -3.41)
 			(stroke
 				(width 0.12)
@@
 		)
 		(fp_line
-			(start -1.695563 2.76)
-			(end 2.76 2.76)
+			(start -3.41 2.345563)
+			(end -2.345563 3.41)
 			(stroke
 				(width 0.12)
@@
 		)
 		(fp_line
-			(start -1.695563 -2.76)
-			(end 2.76 -2.76)
+			(start -3.41 2.345563)
+			(end -3.41 1.06)
 			(stroke
 				(width 0.12)
@@
 		)
 		(fp_line
-			(start -2.76 1.695563)
-			(end -1.695563 2.76)
+			(start -3.41 -2.345563)
+			(end -2.345563 -3.41)
 			(stroke
 				(width 0.12)
@@
 		)
 		(fp_line
-			(start -2.76 1.695563)
-			(end -2.76 1.06)
+			(start -3.41 -2.345563)
+			(end -3.41 -1.06)
 			(stroke
 				(width 0.12)
@@
 		)
 		(fp_line
-			(start -2.76 -1.695563)
-			(end -1.695563 -2.76)
+			(start -4.04375 -2.24125)
+			(end -4.04375 -1.45375)
 			(stroke
 				(width 0.12)
@@
 		)
 		(fp_line
-			(start -2.76 -1.695563)
-			(end -2.76 -1.06)
+			(start -4.4375 -1.8475)
+			(end -3.65 -1.8475)
 			(stroke
 				(width 0.12)
@@
 		)
 		(fp_line
-			(start 3.7 1.05)
-			(end 2.9 1.05)
+			(start 4.8 1.05)
+			(end 3.55 1.05)
 			(stroke
 				(width 0.05)
@@
 		)
 		(fp_line
-			(start 3.7 -1.05)
-			(end 3.7 1.05)
+			(start 4.8 -1.05)
+			(end 4.8 1.05)
 			(stroke
 				(width 0.05)
@@
 		)
 		(fp_line
-			(start 2.9 1.05)
-			(end 2.9 2.9)
+			(start 3.55 1.05)
+			(end 3.55 3.55)
 			(stroke
 				(width 0.05)
@@
 		)
 		(fp_line
-			(start 2.9 -1.05)
-			(end 3.7 -1.05)
+			(start 3.55 -1.05)
+			(end 4.8 -1.05)
 			(stroke
 				(width 0.05)
@@
 		)
 		(fp_line
-			(start 2.9 -2.9)
-			(end 2.9 -1.05)
+			(start 3.55 -3.55)
+			(end 3.55 -1.05)
 			(stroke
 				(width 0.05)
@@
 		)
 		(fp_line
-			(start -1.75 2.9)
-			(end 2.9 2.9)
+			(start -2.4 3.55)
+			(end 3.55 3.55)
 			(stroke
 				(width 0.05)
@@
 		)
 		(fp_line
-			(start -1.75 -2.9)
-			(end 2.9 -2.9)
+			(start -2.4 -3.55)
+			(end 3.55 -3.55)
 			(stroke
 				(width 0.05)
@@
 		)
 		(fp_line
-			(start -2.9 1.75)
-			(end -1.75 2.9)
+			(start -3.55 2.4)
+			(end -2.4 3.55)
 			(stroke
 				(width 0.05)
@@
 		)
 		(fp_line
-			(start -2.9 1.05)
-			(end -2.9 1.75)
+			(start -3.55 1.05)
+			(end -3.55 2.4)
 			(stroke
 				(width 0.05)
@@
 		)
 		(fp_line
-			(start -2.9 -1.05)
-			(end -3.7 -1.05)
+			(start -3.55 -1.05)
+			(end -4.8 -1.05)
 			(stroke
 				(width 0.05)
@@
 		)
 		(fp_line
-			(start -2.9 -1.75)
-			(end -1.75 -2.9)
+			(start -3.55 -2.4)
+			(end -2.4 -3.55)
 			(stroke
 				(width 0.05)
@@
 		)
 		(fp_line
-			(start -2.9 -1.75)
-			(end -2.9 -1.05)
+			(start -3.55 -2.4)
+			(end -3.55 -1.05)
 			(stroke
 				(width 0.05)
@@
 		)
 		(fp_line
-			(start -3.7 1.05)
-			(end -2.9 1.05)
+			(start -4.8 1.05)
+			(end -3.55 1.05)
 			(stroke
 				(width 0.05)
@@
 		)
 		(fp_line
-			(start -3.7 -1.05)
-			(end -3.7 1.05)
+			(start -4.8 -1.05)
+			(end -4.8 1.05)
 			(stroke
 				(width 0.05)
@@
 		)
 		(fp_line
-			(start 2.65 -2.65)
-			(end 2.65 2.65)
+			(start 3.3 -3.3)
+			(end 3.3 3.3)
+			(stroke
+				(width 0.1)
+				(type solid)
+			)
+			(layer "F.Fab")
+		)
+		(fp_line
+			(start -2.3 3.3)
+			(end 3.3 3.3)
 			(stroke
 				(width 0.1)
@@
 		)
 		(fp_line
-			(start -1.65 2.65)
-			(end 2.65 2.65)
+			(start -2.3 -3.3)
+			(end 3.3 -3.3)
 			(stroke
 				(width 0.1)
@@
 		)
 		(fp_line
-			(start -1.65 -2.65)
-			(end 2.65 -2.65)
+			(start -2.389838 -1.645)
+			(end -2.389838 -1.015)
 			(stroke
 				(width 0.1)
@@
 		)
 		(fp_line
-			(start -2.65 1.65)
-			(end -1.65 2.65)
+			(start -2.704838 -1.33)
+			(end -2.074838 -1.33)
 			(stroke
 				(width 0.1)
@@
 		)
 		(fp_line
-			(start -2.65 -1.65)
-			(end -1.65 -2.65)
+			(start -3.3 2.3)
+			(end -2.3 3.3)
 			(stroke
 				(width 0.1)
@@
 		)
 		(fp_line
-			(start -2.65 -1.65)
-			(end -2.65 1.65)
+			(start -3.3 -2.3)
+			(end -2.3 -3.3)
+			(stroke
+				(width 0.1)
+				(type solid)
+			)
+			(layer "F.Fab")
+		)
+		(fp_line
+			(start -3.3 -2.3)
+			(end -3.3 2.3)
 			(stroke
 				(width 0.1)
@@
 		(fp_circle
 			(center 0 0)
-			(end 2.5 0)
+			(end 3.15 0)
 			(stroke
 				(width 0.1)
@@
 		)
 		(fp_text user "${REFERENCE}"
-			(at 0 0 0)
+			(at 0 0 180)
 			(layer "F.Fab")
 			(effects
@@
 		)
 		(pad "1" smd roundrect
-			(at -2.0625 0 180)
-			(size 2.775 1.6)
+			(at -2.8 0 180)
+			(size 3.5 1.6)
 			(layers "F.Cu" "F.Mask" "F.Paste")
 			(roundrect_rratio 0.15625)
@@
 		)
 		(pad "2" smd roundrect
-			(at 2.0625 0 180)
-			(size 2.775 1.6)
+			(at 2.8 0 180)
+			(size 3.5 1.6)
 			(layers "F.Cu" "F.Mask" "F.Paste")
 			(roundrect_rratio 0.15625)
@@
 		)
 		(embedded_fonts no)
-		(model "${KICAD9_3DMODEL_DIR}/Capacitor_SMD.3dshapes/C_Elec_5x5.4.step"
+		(model "${KICAD9_3DMODEL_DIR}/Capacitor_SMD.3dshapes/CP_Elec_6.3x5.4.step"
 			(offset
 				(xyz 0 0 0)
@@
 		(tags "capacitor")
 		(property "Reference" "C102"
-			(at 0 -1.68 0)
+			(at 3.55 0 0)
 			(layer "F.SilkS")
 			(effects
@@
 			)
 		)
-		(property "LSCS#" ""
+		(property "LSCS#" "C114098"
 			(at 0 0 270)
 			(unlocked yes)
@@
 	)
 	(via
+		(at 204.5 80)
+		(size 0.8)
+		(drill 0.4)
+		(layers "F.Cu" "B.Cu")
+		(free yes)
+		(net 2)
+	)
+	(via
 		(at 201.2 103.6)
 		(size 0.8)
@@
 	)
 	(via
+		(at 202 78.5)
+		(size 0.8)
+		(drill 0.4)
+		(layers "F.Cu" "B.Cu")
+		(free yes)
+		(net 2)
+	)
+	(via
 		(at 215.8 91.2)
 		(size 0.8)
@@
 	)
 	(segment
-		(start 206.2 81)
-		(end 203.5 81)
+		(start 201.3 81.5)
+		(end 204.5 78.3)
 		(width 1)
 		(layer "F.Cu")
@@
 	)
 	(segment
-		(start 204.5 77.9)
-		(end 203.5 78.9)
+		(start 207.8 80.04)
+		(end 207.16 80.04)
 		(width 1)
 		(layer "F.Cu")
@@
 	)
 	(segment
-		(start 207.16 80.04)
-		(end 206.2 81)
+		(start 204.5 78.3)
+		(end 204.5 77)
 		(width 1)
 		(layer "F.Cu")
@@
 	)
 	(segment
-		(start 207.8 80.04)
-		(end 207.16 80.04)
+		(start 205.7 81.5)
+		(end 201.3 81.5)
 		(width 1)
 		(layer "F.Cu")
@@
 	)
 	(segment
-		(start 204.5 77)
-		(end 204.5 77.9)
+		(start 207.16 80.04)
+		(end 205.7 81.5)
 		(width 1)
 		(layer "F.Cu")
@@
 		(width 1)
 		(layer "F.Cu")
-		(net 3)
-	)
-	(segment
-		(start 203.5 78.9)
-		(end 203.5 81)
-		(width 1)
-		(layer "F.Cu")
